File: sonda-hx711.kicad_pcb (KiCad board)
At the start: 2 copper layers, 54 parts, among them IC1 ATMEGA328P-A, J1 CONN_01X05, J2 CONN_01X02, J3 CONN_01X02, Q1 BC559, Q2 BC559, SW1 Reset, U1 AP1117-50, U10 HX711, U2 AP1117-33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

Commit message: Laying out board.
Parts:
- moved C9 228.8 mm to (59.5, 46.9), turned to 90 degrees
- moved C6 225.9 mm to (70.6, 47.5)
- moved C8 223.8 mm to (70.6, 49.8)
- moved R4 213.2 mm to (83.1, 49.3), turned to 180 degrees
- moved R5 210.5 mm to (83.1, 46.7), turned to 180 degrees
- moved SW1 195.0 mm to (70.4, 65.8)
- moved C3 189.9 mm to (83.2, 64.0)
- moved Y1 187.4 mm to (63.3, 49.5)
- moved IC1 184.6 mm to (70.0, 56.8), turned to 270 degrees
- moved C10 173.8 mm to (70.1, 42.9), turned to 180 degrees
- moved U3 160.6 mm to (83.7, 56.9), turned to 90 degrees
- moved U5 155.8 mm to (87.6, 36.0)
- moved BT1 114.3 mm to (100.6, 59.2), turned to 90 degrees
Connections:
- IC1 pad 10: /qbar_data -> /qbar_clk
- IC1 pad 11: /qbar_clk -> /angles_data
- IC1 pad 12: Net-(IC1-Pad12) -> /angles_clk
- IC1 pad 14: /1WIRE -> Net-(IC1-Pad14)
- IC1 pad 15: Net-(IC1-Pad15) -> /1WIRE
- IC1 pad 2: /angles_data -> Net-(IC1-Pad2)
- IC1 pad 26: Net-(IC1-Pad26) -> /RTC_INT
- IC1 pad 32: /RTC_INT -> Net-(IC1-Pad32)
- IC1 pad 9: /angles_clk -> /qbar_data
- R3 pad 2: Net-(IC1-Pad12) -> Net-(IC1-Pad13)
Routing:
- net GND: track 63.3 -> 111.8 mm, vias 3 -> 4
- net Net-(BT1-Pad1): track 0.00 -> 20.5 mm
- net /SCL: track 0.00 -> 15.8 mm
- net /SDA: track 0.00 -> 13.8 mm
- net Net-(C9-Pad2): track 0.00 -> 10.5 mm
- net /RTC_INT: track 0.00 -> 9.58 mm
- net Net-(C10-Pad2): track 0.00 -> 5.92 mm
- net +3V3: track 0.00 -> 2.54 mm
- net +5V: track 26.9 -> 27.9 mm

Commit message: Laying out board.
Parts:
- removed C2: 22uF, Capacitors_SMD:CP_Elec_6.3x5.3
- D1: footprint LEDs:LED_D5.0mm -> LEDs:LED_1206_HandSoldering
- moved R3 219.6 mm to (74.4, 45.7)
- moved C7 211.1 mm to (68.6, 74.9), turned to 180 degrees
- moved C5 196.7 mm to (80.3, 28.7), turned to 180 degrees
- moved U2 195.3 mm to (80.3, 36.8), turned to 90 degrees
- moved U1 194.3 mm to (78.5, 70.4), turned to 90 degrees
- moved J3 189.1 mm to (85.1, 78.2)
- moved C4 183.6 mm to (78.2, 78.5), turned to 180 degrees
- moved SW1 181.4 mm to (251.7, 68.1)
- moved L1 180.8 mm to (61.0, 83.8)
- moved U4 180.4 mm to (69.6, 68.1), turned to 270 degrees
- moved C1 174.2 mm to (85.9, 70.6), turned to 90 degrees
- moved J2 162.2 mm to (60.2, 62.0)
- moved D1 159.5 mm to (74.4, 43.4), turned to 180 degrees
- moved J1 149.4 mm to (115.6, 20.3)
- moved R6 44.7 mm to (211.3, 155.2)
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Connections:
- IC1 pad 32: Net-(IC1-Pad32) -> /status_LED
- R3 pad 2: Net-(IC1-Pad13) -> /status_LED
Routing:
- net GND: track 111.8 -> 128.1 mm, vias 4 -> 7
- net +BATT: track 0.00 -> 10.4 mm
- net Net-(C10-Pad2): track 5.92 -> 12.9 mm
- net Net-(C9-Pad2): track 10.5 -> 9.35 mm
